File: RPI5-SDexpress-Hat.kicad_pcb (KiCad board)
At the start: 4 copper layers, 26.4 x 56 mm, 51 parts, among them J1 Conn_01x16_Shielded, J11 10102166A812A, J2 Conn_01x04_Shielded, J3 Conn_01x04_Shielded, J5 Conn_02x03_Odd_Even, SW1 SW_Push, U2 STM8S003F3P, U3 LP5907MFX-3.3, U4 TCA9406DC, U5 PAM2306AYPKE

Commit message: Adding BOM, clean up SCH, update FPC connector BOM
Parts:
- J1: value Conn_01x16_Shielded -> FH12A-16S-0.5SH
Changed lines of the file:
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@@
 			)
 		)
-		(property "Value" "Conn_01x16_Shielded"
+		(property "Value" "FH12A-16S-0.5SH"
 			(at 0 5.6 90)
 			(layer "F.Fab")
